File: hardware/fk-databoat.kicad_pcb (KiCad board)
At the start: 2 copper layers, 96.5 x 81.3 mm, 17 parts, among them P1 CONN_01X03, P2 CONN_01X03, P3 CONN_01X03, P4 CONN_01X03, P5 CONN_01X03, U1 VISO, U10 SERIAL_PORT_EXPANDER, U11 ATLAS_SENSOR, U12 ULTIMATE_GPS, U2 FEATHER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

Commit message: Starting to lay down traces.
Parts:
- moved U10 3.59 mm to (208.3, 127.0), turned to 180 degrees
Connections:
- U11 pad 2: /EC_RX -> /EC_TX
Routing:
- net /ISO_V: track 0.00 -> 128.4 mm
- net /ISO_GND: track 0.00 -> 47.5 mm
- net /SPE_ISO_TX3: track 0.00 -> 21.3 mm
- net /SPE_ISO_RX3: track 0.00 -> 21.2 mm
- net /SPE_ISO_TX1: track 0.00 -> 16.2 mm
- net /SPE_ISO_RX1: track 0.00 -> 16.2 mm
- net /EC_RX: track 0.00 -> 14.6 mm
- net /EC_TX: track 0.00 -> 14.6 mm
- net +3V3: track 0.00 -> 12.7 mm
- net /SPE_ISO_TX0: track 0.00 -> 12.0 mm
- net /SPE_ISO_RX0: track 0.00 -> 12.0 mm
- added copper zone on B.Cu, net /ISO_GND
- added copper zone on B.Cu, net GND

Commit message: More routing/laying out.
Parts:
- moved U8 4.83 mm to (226.3, 129.8)
Routing:
- net /SCL: track 0.00 -> 102.1 mm, vias 0 -> 1
- net /SDA: track 0.00 -> 98.3 mm, vias 0 -> 1
- net /SPE_NOR_TX: track 0.00 -> 61.8 mm, vias 0 -> 1
- net /SPE_ISO_SEL_0: track 0.00 -> 59.0 mm
- net /SPE_NOR_RX: track 0.00 -> 58.4 mm, vias 0 -> 1
- net /SPE_ISO_SEL_1: track 0.00 -> 55.3 mm, vias 0 -> 1
- net /ISO_GND: track 47.5 -> 0.00 mm
- net /SPE_ISO_TX2: track 0.00 -> 29.6 mm
- net /SPE_ISO_RX2: track 0.00 -> 29.0 mm
- net /VLOAD: track 0.00 -> 25.4 mm, vias 0 -> 1
- net /INT_TX: track 0.00 -> 23.1 mm
- net /INT_RX: track 0.00 -> 23.0 mm
- net /SPE_ISO_RX: track 0.00 -> 18.0 mm
- net +3V3: track 12.7 -> 27.9 mm
- net /SPE_NOR_SEL_0: track 0.00 -> 12.7 mm, vias 0 -> 1

Commit message: Last of the routing. Gonna do the cap on the solar charger now.
Connections:
- U1 pad 10: /INT_SEL_0 -> /INT_SEL_1
- U3 pad 4: /INT_SEL_0 -> /INT_SEL_1
Routing:
- net +3V3: track 27.9 -> 195.7 mm
- net /GPS_TX: track 0.00 -> 68.1 mm
- net /GPS_RX: track 0.00 -> 66.3 mm
- net /B+: track 0.00 -> 44.4 mm
- net /B-: track 0.00 -> 43.4 mm
- net /SPE_NOR_SEL_0: track 12.7 -> 53.4 mm
- net /INT_SEL_0: track 0.00 -> 40.5 mm, vias 0 -> 1
- net /INT_SEL_1: track 0.00 -> 40.5 mm, vias 0 -> 1
- net GND: track 0.00 -> 37.4 mm, vias 0 -> 6
- net /VLOAD: track 25.4 -> 52.0 mm
- net /SPE_ISO_TX: track 0.00 -> 17.8 mm, vias 0 -> 1
- net /SPE_ISO_SEL_1: track 55.3 -> 59.9 mm
- net /SPE_NOR_TX: track 61.8 -> 64.5 mm
- net /SPE_NOR_RX: track 58.4 -> 61.1 mm
- net /SPE_ISO_SEL_0: track 59.0 -> 61.5 mm
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- added copper zone on F.Cu, net GND

Commit message: Add solar charger that pulls out some connections to slim things up.
Parts:
- added J1: CONN_01X02, Socket_Strips:Socket_Strip_Straight_1x02_Pitch2.54mm, F.Cu at (222.0, 139.7)
- added J2: CONN_01X02, Socket_Strips:Socket_Strip_Straight_1x02_Pitch2.54mm, F.Cu at (222.0, 128.8)
- U8: value adafruit-solar-charger -> adafruit-solar-charger-with-cap; footprint conservify:adafruit-solar-charger -> conservify:adafruit-solar-charger-with-cap
- moved U8 0.25 mm to (226.1, 129.8)
Routing:
- net Net-(J2-Pad2): track 0.00 -> 25.4 mm
- net Net-(J2-Pad1): track 0.00 -> 20.4 mm
- net Net-(J1-Pad2): track 0.00 -> 12.7 mm
- net Net-(J1-Pad1): track 0.00 -> 10.5 mm
- net +3V3: track 195.7 -> 197.2 mm
Other:
- board text added: "4700uF"
- board text added: "DO"
- board text added: "EC"
- board text added: "GPS"
- board text added: "ORP"
- board text added: "PH"
- board text added: "SOLAR"
- board text added: "TEMP"
